File: 33reg.kicad_pcb (KiCad board)
At the start: 2 copper layers, 7 parts, among them P1 TST, P2 TST, P3 TST, U1 AAT1110IJS-3.3-T1

Commit message: pcb done, add gerbers+drill
Parts:
- added GND: TST, TEST_0.100, F.Cu at (207.0, 134.6)
- moved C1 5.18 mm to (196.3, 135.5), turned to 180 degrees
- moved C2 5.08 mm to (203.2, 134.6), turned to 90 degrees
- renumbered P3 to +3.3V, P1 to +5V, P2 to GND
Routing:
- net +3.3v: track 0.00 -> 15.1 mm
- net +5v: track 0.00 -> 13.2 mm
- net N-000002: track 0.00 -> 9.29 mm, vias 0 -> 2
- net GND: track 0.00 -> 4.91 mm, vias 0 -> 3
- added copper zone on B.Cu, net GND
- added copper zone on F.Cu, net GND
Other:
- board outline added: 16.8 x 12.1 mm
- net class Default: clearance 0.254 -> 0.1524
- rule trace_clearance: 0.254 -> 0.1524
- rule trace_min: 0.254 -> 0.1524
- board text added: "+5v to +3.3v buck v0.1 oct-2013 github.com/noahp/3_3swreg"
- board text added: "."
